File: mmms_sorter_schema/mmms_sorter_schema.kicad_pcb (KiCad board)
At the start: 2 copper layers, 13 parts, among them M1 Director Servo, M2 Latch Servo, U1 L7805, U2 APDS-9960, U3 ULN2003

Commit message: Refine schema and software
Parts:
- removed C1: 0,33uF, Capacitor_THT:CP_Radial_D4.0mm_P1.50mm
- removed C2: 0,1uF, Capacitor_THT:CP_Radial_D4.0mm_P1.50mm
- removed the REF** at (116.8, 128.3)
- removed the REF** at (149.9, 71.1)
- removed the REF** at (116.8, 71.1)
- removed U1: L7805, Package_TO_SOT_THT:TO-220-3_Vertical
- added REF**: PinHeader_1x02_P2.54mm_Vertical, Connector_PinHeader_2.54mm:PinHeader_1x02_P2.54mm_Vertical, F.Cu at (173.4, 103.5)
- R1: footprint Resistor_THT:R_Axial_DIN0204_L3.6mm_D1.6mm_P2.54mm_Vertical -> Resistor_THT:R_Axial_DIN0204_L3.6mm_D1.6mm_P7.62mm_Horizontal
- moved U2 41.0 mm to (175.9, 69.8), turned to 180 degrees
- moved M2 36.5 mm to (113.7, 66.0), turned to 180 degrees
- moved D1 36.4 mm to (175.9, 85.1)
- moved R1 32.0 mm to (160.7, 95.2)
- moved A1 29.5 mm to (130.2, 58.4)
- moved M1 27.9 mm to (113.7, 81.3), turned to 0 degrees
- moved U3 5.43 mm to (131.4, 109.2), turned to 90 degrees
Connections:
- net 3v3 renamed Net-(A1-Pad17)
- net 5V renamed +5V
- M1 pad 1: Net-(A1-Pad8) -> Net-(A1-Pad9)
- M2 pad 1: Net-(A1-Pad9) -> Net-(A1-Pad8)
- U2 pad 3: Net-(U2-Pad3) -> SDA
- U2 pad 4: SDA -> SCL
- U2 pad 5: SCL -> (no net)
- U3 pad 2: Net-(A1-Pad14) -> Net-(A1-Pad13)
- U3 pad 3: Net-(A1-Pad13) -> Net-(A1-Pad14)
Routing:
- net GND: track 100.1 -> 241.4 mm
- net +5V: track 74.1 -> 151.3 mm
- net Net-(A1-Pad9): track 47.6 -> 17.6 mm
- net Net-(A1-Pad12): track 5.61 -> 28.6 mm
- net Net-(A1-Pad10): track 25.0 -> 42.8 mm
- net Net-(A1-Pad14): track 10.3 -> 22.5 mm
- net SCL: track 25.7 -> 35.2 mm
- net Net-(A1-Pad13): track 16.1 -> 25.6 mm
- net External5V: track 7.40 -> 0.00 mm
- net SDA: track 29.3 -> 35.2 mm
- net Net-(D1-Pad2): track 18.8 -> 15.2 mm
- net Net-(A1-Pad15): track 16.4 -> 18.9 mm
- net Net-(A1-Pad17): track 46.6 -> 47.9 mm
- net Net-(A1-Pad8): track 21.7 -> 20.7 mm
- added copper zone on F.Cu, net GND
Other:
- board text added: "Dawid Dziedzic Sorter MMMS 2021 v0.2"
