File: mmms_sorter_schema/mmms_sorter_schema.sch (KiCad schematic (older format))
At the start: 10 parts, among them M1 Director Servo, M2 Latch Servo, U1 L7805, U2 APDS-9960, U3 ULN2003

Commit message: Refine schema and software
Parts:
- removed C1: 0,33uF, Capacitor_THT:CP_Radial_D4.0mm_P1.50mm, symbol Device:C
- removed C2: 0,1uF, Capacitor_THT:CP_Radial_D4.0mm_P1.50mm, symbol Device:C
- removed U1: L7805, Package_TO_SOT_THT:TO-220-3_Vertical, symbol Regulator_Linear:L7805
- R1: footprint Resistor_THT:R_Axial_DIN0204_L3.6mm_D1.6mm_P2.54mm_Vertical -> Resistor_THT:R_Axial_DIN0204_L3.6mm_D1.6mm_P7.62mm_Horizontal
Connections:
- net at A1.13 (D10): now also U3.2 (I2); no longer U3.3 (I3)
- net at A1.14 (D11): now also U3.3 (I3); no longer U3.2 (I2)
- net at A1.8 (D5): now also M2.1 (PWM); no longer M1.1 (PWM)
- net at A1.9 (D6): now also M1.1 (PWM); no longer M2.1 (PWM)
- net 3v3: no longer names the net of A1.17 (3V3), U2.2 (Vcc)
- net 5V renamed +5V
Changed lines of the file:
@@
 P 7450 1850
 F 0 "U2" H 7800 2250 50  0001 R CNN
-F 1 "APDS-9960" H 7950 2150 50  0000 R CNN
+F 1 "APDS-9960" H 8000 2150 50  0000 R CNN
 F 2 "Connector_PinHeader_2.54mm:PinHeader_1x06_P2.54mm_Vertical" H 7450 1850 50  0001 C CNN
 F 3 "" H 7450 1850 50  0001 C CNN
@@
 	-1   0    0    -1
 $EndComp
-Text GLabel 7450 1450 1    50   UnSpc ~ 0
-3v3
-Text GLabel 3750 1500 1    50   UnSpc ~ 0
-3v3
 $Comp
 L Device:R R1
@@
 F 0 "R1" V 6793 2550 50  0001 C CNN
 F 1 "180R" V 6885 2550 50  0000 C CNN
-F 2 "Resistor_THT:R_Axial_DIN0204_L3.6mm_D1.6mm_P2.54mm_Vertical" V 6930 2550 50  0001 C CNN
+F 2 "Resistor_THT:R_Axial_DIN0204_L3.6mm_D1.6mm_P7.62mm_Horizontal" V 6930 2550 50  0001 C CNN
 F 3 "~" H 7000 2550 50  0001 C CNN
 	1    7000 2550
@@
 $EndComp
 Wire Wire Line
-	5050 2800 6850 2800
+	5050 2750 6850 2750
 Wire Notes Line
 	7900 1150 6700 1150
@@
 	1    0    0    -1
 $EndComp
-Text GLabel 3950 1500 1    50   UnSpc ~ 0
-5V
-Text GLabel 5550 2550 0    50   UnSpc ~ 0
-5V
-Text GLabel 5450 2100 0    50   UnSpc ~ 0
-5V
-Wire Wire Line
-	4350 2550 5200 2550
-Wire Wire Line
-	5200 2450 5600 2450
-Wire Wire Line
-	5200 2550 5200 2450
-Wire Wire Line
-	4350 2450 4900 2450
-Wire Wire Line
-	4900 2450 4900 2000
-Wire Wire Line
-	4900 2000 5500 2000
-Wire Wire Line
-	5450 2100 5500 2100
-Wire Wire Line
-	5450 2200 5500 2200
-Wire Wire Line
-	5550 2550 5600 2550
-Wire Wire Line
-	5550 2650 5600 2650
 Wire Wire Line
 	3750 3550 3750 3600
 Wire Wire Line
-	6850 2550 6850 2800
-Wire Wire Line
-	3750 1550 3750 1500
+	6850 2550 6850 2750
 Wire Wire Line
 	3950 1550 3950 1500
 Wire Wire Line
-	7450 1500 7450 1450
-$Comp
-L Regulator_Linear:L7805 U1
-U 1 1 609525EC
-P 5500 1050
-F 0 "U1" H 5500 1292 50  0001 C CNN
-F 1 "L7805" H 5500 1201 50  0000 C CNN
-F 2 "Package_TO_SOT_THT:TO-220-3_Vertical" H 5525 900 50  0001 L CIN
-F 3 "http://www.st.com/content/ccc/resource/technical/document/datasheet/41/4f/b3/b0/12/d4/47/88/CD00000444.pdf/files/CD00000444.pdf/jcr:content/translations/en.CD00000444.pdf" H 5500 1000 50  0001 C CNN
-	1    5500 1050
-	1    0    0    -1
-$EndComp
-$Comp
-L Device:C C2
-U 1 1 609580F1
-P 6000 1350
-F 0 "C2" H 6115 1396 50  0001 L CNN
-F 1 "0,1uF" H 6115 1350 50  0000 L CNN
-F 2 "Capacitor_THT:CP_Radial_D4.0mm_P1.50mm" H 6038 1200 50  0001 C CNN
-F 3 "~" H 6000 1350 50  0001 C CNN
-	1    6000 1350
-	1    0    0    -1
-$EndComp
-Connection ~ 5500 1500
-Wire Wire Line
-	5800 1050 6000 1050
-Wire Wire Line
-	6000 1500 5500 1500
-$Comp
-L Device:C C1
-U 1 1 609660FB
-P 4950 1350
-F 0 "C1" H 5065 1396 50  0001 L CNN
-F 1 "0,33uF" H 5065 1350 50  0000 L CNN
-F 2 "Capacitor_THT:CP_Radial_D4.0mm_P1.50mm" H 4988 1200 50  0001 C CNN
-F 3 "~" H 4950 1350 50  0001 C CNN
-	1    4950 1350
-	1    0    0    -1
-$EndComp
-Text GLabel 6200 1050 2    50   UnSpc ~ 0
-5V
-Wire Wire Line
-	6200 1050 6000 1050
-Connection ~ 6000 1050
-Text GLabel 4850 1050 0    50   UnSpc ~ 0
-External5V
-Wire Wire Line
-	4950 1500 5500 1500
-Wire Wire Line
-	4850 1050 4950 1050
-Connection ~ 4950 1050
-Wire Wire Line
-	4950 1050 5200 1050
-Wire Wire Line
-	5500 1350 5500 1500
-Wire Wire Line
-	5500 1500 5500 1600
-Wire Wire Line
-	6000 1050 6000 1200
-Wire Wire Line
-	4950 1050 4950 1200
-Wire Wire Line
-	5050 2650 5050 2800
+	5050 2650 5050 2750
 Wire Wire Line
 	4350 2650 5050 2650
@@
 $EndComp
 $Comp
-L power:GND #PWR0101
-U 1 1 6092908C
-P 5500 1600
-F 0 "#PWR0101" H 5500 1350 50  0001 C CNN
-F 1 "GND" H 5505 1427 50  0000 C CNN
-F 2 "" H 5500 1600 50  0001 C CNN
-F 3 "" H 5500 1600 50  0001 C CNN
-	1    5500 1600
-	1    0    0    -1
-$EndComp
-$Comp
 L power:GND #PWR0102
 U 1 1 6092AEEC
@@
 L power:GND #PWR0103
 U 1 1 6092B683
-P 5550 2650
-F 0 "#PWR0103" H 5550 2400 50  0001 C CNN
-F 1 "GND" V 5555 2522 50  0000 R CNN
-F 2 "" H 5550 2650 50  0001 C CNN
-F 3 "" H 5550 2650 50  0001 C CNN
-	1    5550 2650
+P 5500 2650
+F 0 "#PWR0103" H 5500 2400 50  0001 C CNN
+F 1 "GND" V 5505 2522 50  0000 R CNN
+F 2 "" H 5500 2650 50  0001 C CNN
+F 3 "" H 5500 2650 50  0001 C CNN
+	1    5500 2650
 	0    1    1    0
 $EndComp
@@
 L power:GND #PWR0104
 U 1 1 6092BD9F
-P 5450 2200
-F 0 "#PWR0104" H 5450 1950 50  0001 C CNN
-F 1 "GND" V 5455 2072 50  0000 R CNN
-F 2 "" H 5450 2200 50  0001 C CNN
-F 3 "" H 5450 2200 50  0001 C CNN
-	1    5450 2200
+P 5400 2200
+F 0 "#PWR0104" H 5400 1950 50  0001 C CNN
+F 1 "GND" V 5405 2072 50  0000 R CNN
+F 2 "" H 5400 2200 50  0001 C CNN
+F 3 "" H 5400 2200 50  0001 C CNN
+	1    5400 2200
 	0    1    1    0
 $EndComp
@@
 Wire Wire Line
 	7450 2450 7450 2550
-Wire Wire Line
-	4350 2850 5350 2850
-Wire Wire Line
-	5350 2850 5350 3300
-Wire Wire Line
-	5300 3400 5350 3400
-Wire Wire Line
-	5250 3500 5350 3500
-Wire Wire Line
-	5200 3600 5350 3600
 $Comp
 L customs:ULN2003 U3
@@
 	1    0    0    -1
 $EndComp
-Text GLabel 5750 3050 1    50   UnSpc ~ 0
-5V
-Wire Wire Line
-	5750 3050 5750 3100
 Wire Wire Line
 	5750 3800 5750 3850
-Wire Wire Line
-	5300 3400 5300 3050
-Wire Wire Line
-	5300 3050 4350 3050
-Wire Wire Line
-	4350 2950 5250 2950
-Wire Wire Line
-	5250 2950 5250 3500
-Wire Wire Line
-	4350 3150 5200 3150
-Wire Wire Line
-	5200 3150 5200 3600
+$Comp
+L power:+5V #PWR01
+U 1 1 6096B7CF
+P 3950 1500
+F 0 "#PWR01" H 3950 1350 50  0001 C CNN
+F 1 "+5V" H 3965 1673 50  0000 C CNN
+F 2 "" H 3950 1500 50  0001 C CNN
+F 3 "" H 3950 1500 50  0001 C CNN
+	1    3950 1500
+	1    0    0    -1
+$EndComp
+$Comp
+L power:+5V #PWR02
+U 1 1 6096C377
+P 5400 2100
+F 0 "#PWR02" H 5400 1950 50  0001 C CNN
+F 1 "+5V" V 5415 2228 50  0000 L CNN
+F 2 "" H 5400 2100 50  0001 C CNN
+F 3 "" H 5400 2100 50  0001 C CNN
+	1    5400 2100
+	0    -1   -1   0
+$EndComp
+$Comp
+L power:+5V #PWR03
+U 1 1 60972E13
+P 5500 2550
+F 0 "#PWR03" H 5500 2400 50  0001 C CNN
+F 1 "+5V" V 5515 2678 50  0000 L CNN
+F 2 "" H 5500 2550 50  0001 C CNN
+F 3 "" H 5500 2550 50  0001 C CNN
+	1    5500 2550
+	0    -1   -1   0
+$EndComp
+Wire Wire Line
+	5500 2650 5600 2650
+Wire Wire Line
+	5500 2550 5600 2550
+Wire Wire Line
+	5400 2200 5500 2200
+Wire Wire Line
+	5400 2100 5500 2100
+Wire Wire Line
+	7450 1200 3750 1200
+Wire Wire Line
+	3750 1200 3750 1550
+Wire Wire Line
+	7450 1200 7450 1500
+$Comp
+L power:+5V #PWR04
+U 1 1 60981275
+P 5750 3000
+F 0 "#PWR04" H 5750 2850 50  0001 C CNN
+F 1 "+5V" H 5765 3173 50  0000 C CNN
+F 2 "" H 5750 3000 50  0001 C CNN
+F 3 "" H 5750 3000 50  0001 C CNN
+	1    5750 3000
+	1    0    0    -1
+$EndComp
+Wire Wire Line
+	5750 3000 5750 3100
+Wire Wire Line
+	4350 2450 5600 2450
+Wire Wire Line
+	4350 2550 4800 2550
+Wire Wire Line
+	4800 2550 4800 2000
+Wire Wire Line
+	4800 2000 5500 2000
+Wire Wire Line
+	5350 3300 4850 3300
+Wire Wire Line
+	4850 3300 4850 2850
+Wire Wire Line
+	4850 2850 4350 2850
+Wire Wire Line
+	4350 2950 4800 2950
+Wire Wire Line
+	4800 2950 4800 3400
+Wire Wire Line
+	4800 3400 5350 3400
+Wire Wire Line
+	4350 3050 4750 3050
+Wire Wire Line
+	4750 3050 4750 3500
+Wire Wire Line
+	4750 3500 5350 3500
+Wire Wire Line
+	4350 3150 4700 3150
+Wire Wire Line
+	4700 3150 4700 3600
+Wire Wire Line
+	4700 3600 5350 3600
 $EndSCHEMATC
